File: PCB_Robot/PCB_Robot.kicad_sch (KiCad schematic)
At the start: 15 parts, among them J1 UART, J2 Alimentacion, J3 MotorL, J4 MotorR, U1 ESP32-WROOM-E, U2 TB6612FNG, U3 BMI160

Commit message: PCB Actualizda
Connections:
- no-connect marks 6 -> 18
Changed lines of the file:
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@@
+	)
+	(no_connect
+		(at 49.53 73.66)
+	)
+	(no_connect
+		(at 115.57 73.66)
+	)
+	(no_connect
+		(at 49.53 71.12)
+	)
+	(no_connect
+		(at 115.57 55.88)
+	)
+	(no_connect
+		(at 49.53 60.96)
 	)
 	(no_connect
@@
 	)
 	(no_connect
+		(at 115.57 78.74)
+	)
+	(no_connect
+		(at 115.57 76.2)
+	)
+	(no_connect
+		(at 49.53 66.04)
+	)
+	(no_connect
 		(at 63.5 161.29)
+	)
+	(no_connect
+		(at 49.53 76.2)
+	)
+	(no_connect
+		(at 49.53 78.74)
 	)
 	(no_connect
@@
 	)
 	(no_connect
+		(at 115.57 71.12)
+	)
+	(no_connect
 		(at 63.5 153.67)
 	)
 	(no_connect
+		(at 115.57 58.42)
+	)
+	(no_connect
